File: 35keypad.kicad_pcb (KiCad board)
At the start: 2 copper layers, 143.4 x 105.4 mm, 104 parts, among them J1 USB_C_Receptacle_USB2.0, SW1 SW_SPST, SW10 KEY_10_21, SW11 KEY_10_21, SW12 KEY_10_21, SW13 KEY_3_02, SW14 KEY_7_12, SW15 KEY_11_22, SW16 KEY_11_22, SW17 KEY_11_22, SW18 KEY_4_03, SW19 KEY_8_13, SW2 SW_SPST, SW20 KEY_12_23, SW21 KEY_12_23, SW22 KEY_12_23, SW23 KEY_4_03, SW24 KEY_4_03, SW25 KEY_4_03, SW26 KEY_4_03, SW27 KEY_4_03, SW28 KEY_4_03, SW29 KEY_8_13, SW3 KEY_1_00, SW30 KEY_12_23, SW31 KEY_12_23, SW32 KEY_12_23, SW33 KEY_4_03, SW34 KEY_4_03, SW35 KEY_4_03, SW36 KEY_4_03, SW37 KEY_4_03, SW4 KEY_5_10, SW5 KEY_9_20, SW6 KEY_9_20, SW7 KEY_9_20, SW8 KEY_2_01, SW9 KEY_6_11, U1 W25Q128JVS, U2 RP2040, U3 NCP1117-3.3_SOT223, Y1 12MHz

Commit message: files: add finished pcb layout
Parts:
- C5, C8: value 10u -> 1u; footprint Capacitor_SMD:C_0603_1608Metric -> Capacitor_SMD:C_0402_1005Metric
- D1, D10, D11, D12, D13, D14, D15, D16, D17, D18, D19, D2, D20, D21, D22, D23, D24, D25, D26, D27, D28, D29, D3, D30, D31, D32, D33, D34, D35, D4, D5, D6, D7, D8, D9: footprint Diode_SMD:D_SOD-123 -> Diode_SMD:D_SOD-323
- U3: footprint Package_TO_SOT_SMD:SOT-223-3_TabPin2 -> Package_TO_SOT_SMD:SOT-23-3
- moved D35 202.1 mm to (57.9, 133.1), turned to -90 degrees
- moved D34 196.9 mm to (57.9, 114.0), turned to -90 degrees
- moved D33 192.9 mm to (57.9, 95.0), turned to -90 degrees
- moved D30 191.7 mm to (76.9, 133.1), turned to -90 degrees
- moved D32 190.2 mm to (57.8, 75.9), turned to -90 degrees
- moved D31 188.6 mm to (57.9, 56.9), turned to -90 degrees
- moved D29 184.9 mm to (76.9, 114.0), turned to -90 degrees
- moved D28 167.2 mm to (76.9, 95.0), turned to -90 degrees
- moved D25 166.8 mm to (95.9, 133.1), turned to -90 degrees
- moved D27 164.6 mm to (76.9, 75.9), turned to -90 degrees
- moved D26 163.5 mm to (76.9, 56.9), turned to -90 degrees
- moved D24 159.5 mm to (96.0, 114.0), turned to -90 degrees
- moved D23 153.5 mm to (96.0, 95.0), turned to -90 degrees
- moved D22 148.9 mm to (96.0, 75.9), turned to -90 degrees
- moved D20 142.1 mm to (115.0, 133.1), turned to -90 degrees
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Connections:
- U2 pad 13: /COL_4 -> /COL_3
- U2 pad 14: /COL_3 -> unconnected-(U2-GPIO11-Pad14)
- U2 pad 15: /COL_2 -> unconnected-(U2-GPIO12-Pad15)
- U2 pad 16: /ROW_4 -> unconnected-(U2-GPIO13-Pad16)
- U2 pad 17: /ROW_3 -> unconnected-(U2-GPIO14-Pad17)
- U2 pad 2: unconnected-(U2-GPIO0-Pad2) -> /COL_6
- U2 pad 28: unconnected-(U2-GPIO17-Pad28) -> /ROW_4
- U2 pad 29: unconnected-(U2-GPIO18-Pad29) -> /ROW_3
- U2 pad 32: unconnected-(U2-GPIO21-Pad32) -> /ROW_1
- U2 pad 34: /ROW_1 -> /COL_2
- U2 pad 35: /COL_0 -> /COL_1
- U2 pad 36: /COL_1 -> /COL_0
- U2 pad 5: unconnected-(U2-GPIO3-Pad5) -> /COL_5
- U2 pad 7: /COL_6 -> unconnected-(U2-GPIO5-Pad7)
- U2 pad 8: /COL_5 -> /COL_4
Routing:
- net /ROW_4: track 0.00 -> 190.8 mm, vias 0 -> 14
- net /ROW_3: track 0.00 -> 173.5 mm, vias 0 -> 14
- net /ROW_2: track 0.00 -> 155.3 mm, vias 0 -> 14
- net /ROW_1: track 0.00 -> 144.3 mm, vias 0 -> 12
- net /COL_6: track 0.00 -> 137.7 mm, vias 0 -> 4
- net /ROW_0: track 0.00 -> 136.0 mm, vias 0 -> 6
- net /COL_0: track 0.00 -> 133.7 mm, vias 0 -> 4
- net /COL_5: track 0.00 -> 123.0 mm, vias 0 -> 2
- net /COL_1: track 0.00 -> 111.3 mm, vias 0 -> 2
- net /COL_4: track 0.00 -> 102.8 mm, vias 0 -> 4
- net /COL_2: track 0.00 -> 92.0 mm, vias 0 -> 2
- net /COL_3: track 0.00 -> 85.8 mm, vias 0 -> 2
- net +3V3: track 0.00 -> 57.4 mm, vias 0 -> 4
- net Net-(SW1-B): track 0.00 -> 30.0 mm
- net GND: track 0.00 -> 29.3 mm, vias 0 -> 30
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- added copper zone on F.Cu, net +1V1
- added copper zone on F.Cu, net GND
- added copper zone on F.Cu, net VBUS
Other:
- board text added: "BOOT"
- board text added: "RESET"
