File: v1/35keypad.kicad_pcb (KiCad board)
At the start: 2 copper layers, 143.4 x 105.4 mm, 104 parts, among them J1 USB_C_Receptacle_USB2.0, SW1 SW_SPST, SW10 KEY_10_21, SW11 KEY_10_21, SW12 KEY_10_21, SW13 KEY_3_02, SW14 KEY_7_12, SW15 KEY_11_22, SW16 KEY_11_22, SW17 KEY_11_22, SW18 KEY_4_03, SW19 KEY_8_13, SW2 SW_SPST, SW20 KEY_12_23, SW21 KEY_12_23, SW22 KEY_12_23, SW23 KEY_4_03, SW24 KEY_4_03, SW25 KEY_4_03, SW26 KEY_4_03, SW27 KEY_4_03, SW28 KEY_4_03, SW29 KEY_8_13, SW3 KEY_1_00, SW30 KEY_12_23, SW31 KEY_12_23, SW32 KEY_12_23, SW33 KEY_4_03, SW34 KEY_4_03, SW35 KEY_4_03, SW36 KEY_4_03, SW37 KEY_4_03, SW4 KEY_5_10, SW5 KEY_9_20, SW6 KEY_9_20, SW7 KEY_9_20, SW8 KEY_2_01, SW9 KEY_6_11, U1 W25Q128JVS, U2 RP2040, U3 NCP1117-3.3_SOT223, Y1 12MHz

Commit message: refactor: add v1 folder and move files
Other:
- board text added: "Diodes need to be move away from hot swap socket pad 2"
- board text added: "error mcu and capacitors go under hot swap socket"
Changed lines of the file:
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@@
+	)
+	(gr_line
+		(start 143.6116 56.4896)
+		(end 164.7444 35.3568)
+		(stroke
+			(width 2)
+			(type default)
+		)
+		(layer "Cmts.User")
 	)
 	(gr_line
@@
 		(layer "Cmts.User")
 	)
+	(gr_rect
+		(start 132.7404 56.4896)
+		(end 143.6116 67.3608)
+		(stroke
+			(width 2)
+			(type default)
+		)
+		(fill none)
+		(layer "Cmts.User")
+	)
 	(gr_line
 		(start 56.555 145.425)
@@
 				(bold yes)
 			)
+			(justify left bottom)
+		)
+	)
+	(gr_text "Diodes need to be move away \nfrom hot swap socket pad 2"
+		(at 50.4444 39.9288 0)
+		(layer "Cmts.User")
+		(effects
+			(font
+				(size 2 2)
+				(thickness 0.5)
+				(bold yes)
+			)
+			(justify left bottom)
+		)
+	)
+	(gr_text "error\nmcu and capacitors \ngo under hot swap socket"
+		(at 164.7444 35.3568 0)
+		(layer "Cmts.User")
+		(effects
+			(font
+				(size 5 5)
+				(thickness 1)
+				(bold yes)
+			)
